Commit message: added camera_mount urdf

File: braccio_description/urdf/braccio_camera_model.urdf (robot description, URDF)
Before this commit: robot kuka, 9 links, 8 joints
Links:
- removed link camera_mount_base
- added link camera_mount; collision mesh filename=package://braccio_arduino_ros_rviz/stl/geometry.stl scale=0.001 0.001 0.001; visual mesh filename=package://braccio_arduino_ros_rviz/stl/geometry.stl scale=0.001 0.001 0.001
- added link world
Joints:
- removed joint camera_mount_joint
- added joint camera: type fixed, parent world, child base_link, origin xyz=0 0 -1.57079632679 rpy=0 0 0
- added joint world_joint: type fixed, parent world, child base_link, origin xyz=0.0 0.0 0.0 rpy=0.0 0.0 0.0

File: braccio_description/urdf/braccio_full.urdf (robot description, URDF)
Before this commit: robot kuka, 9 links, 8 joints
Links:
- added link camera_mount_pillar, mass 1.0; collision box size=0.01 0.1 0.5; visual box size=0.01 0.1 0.5
- added link camera_top_link; collision box size=0.1 0.5 0.1; visual box size=0.1 0.5 0.01
- added link world
- link camera_mount_base: mass None -> 1.0; geometry collision box size=0.1 0.5 0.01; visual box size=0.1 0.5 0.01
Joints:
- removed joint camera_mount_joint
- added joint mount_pillar_joint: type fixed, parent camera_mount_base, child camera_mount_pillar, origin xyz=0.0 0.005 0.245 rpy=0 0 0
- added joint pillar_top_joint: type fixed, parent camera_mount_base, child camera_top_link, origin xyz=0.0 0.01 0.0 rpy=0 0 0
- added joint world_joint: type fixed, parent world, child base_link, origin xyz=0.0 0.0 0.0 rpy=0.0 0.0 0.0

File: braccio_description/urdf/xacros/_d435.urdf.xacro (robot description, xacro)
@@ -32,15 +32,15 @@
     </material>
     <!-- camera body, with origin at bottom screw mount -->
+    <link name="${name}_bottom_screw_frame"/>
     <!-- <joint name="${name}_joint" type="fixed">
       <xacro:insert_block name="origin" />
       <parent link="${parent}"/>
       <child link="${name}_bottom_screw_frame" />
-    </joint>
-    <link name="${name}_bottom_screw_frame"/>
+    </joint> -->
     <joint name="${name}_link_joint" type="fixed">
       <origin xyz="0 ${d435_cam_depth_py} ${d435_cam_depth_pz}" rpy="0 0 0"/>
       <parent link="${name}_bottom_screw_frame"/>
       <child link="${name}_link" />
-    </joint> -->
+    </joint>
     <link name="${name}_link">
       <visual>
@@ -121,6 +121,6 @@
     <xacro:gazebo_d435 camera_name="${name}" reference_link="${name}_link" topics_ns="${topics_ns}" depth_optical_frame="${name}_depth_optical_frame" color_optical_frame="${name}_color_optical_frame" infrared1_optical_frame="${name}_left_ir_optical_frame" infrared2_optical_frame="${name}_right_ir_optical_frame" publish_pointcloud="${publish_pointcloud}"/>
   </xacro:macro>
-    <xacro:sensor_d435 parent='world'>
-          <origin xyz="0.0 0.0 0.0" rpy="0.0 0.0 0.0" />
+    <xacro:sensor_d435 parent="world">
+          <origin xyz="0.0 0.0 0.5" rpy="0.0 0.0 0.0" />
     </xacro:sensor_d435>
 </robot>
