Commit message: tried spawn world with camera mount

File: braccio_description/urdf/braccio_model.urdf (robot description, URDF)
Before this commit: robot kuka, 9 links, 8 joints
Joints:
- joint camera_mount_joint: origin xyz=0.0 0.0 0.0 rpy=0.0 0.0 0.0 -> xyz=0.0 0.0 0.01 rpy=0.0 0.0 0.0

Commit message: added mounting mesh

File: braccio_description/urdf/braccio_model.urdf (robot description, URDF)
Before this commit: robot kuka, 9 links, 8 joints
Links:
- removed link camera_mount_base
- added link mount
Joints:
- joint camera_mount_joint: origin xyz=0.0 0.0 0.01 rpy=0.0 0.0 0.0 -> xyz=0.0 0.0 0.00 rpy=0.0 0.0 0.0; parent camera_mount_base -> mount

File: braccio_description/urdf/xacros/_d435.urdf.xacro (robot description, xacro)
@@ -121,6 +121,7 @@
     <xacro:gazebo_d435 camera_name="${name}" reference_link="${name}_link" topics_ns="${topics_ns}" depth_optical_frame="${name}_depth_optical_frame" color_optical_frame="${name}_color_optical_frame" infrared1_optical_frame="${name}_left_ir_optical_frame" infrared2_optical_frame="${name}_right_ir_optical_frame" publish_pointcloud="${publish_pointcloud}"/>
   </xacro:macro>
-    <xacro:sensor_d435 parent="world">
-          <origin xyz="0.0 0.0 0.5" rpy="0.0 0.0 0.0" />
+    <xacro:sensor_d435 parent="mount">
+          <!-- <origin xyz="0.0 0.0 0.5" rpy="0.0 0.0 0.0" /> -->
+          <origin xyz="0.0857 0.0000476009 -0.273184" rpy="0.0 0.0 0.0" />
     </xacro:sensor_d435>
 </robot>

Commit message: added full system xacro

File: braccio_description/urdf/braccio_model.urdf (robot description, URDF)
Before this commit: robot kuka, 9 links, 8 joints
Links:
- removed link mount
- added link world
Joints:
- joint camera_mount_joint: parent mount -> world; type continuous -> fixed

File: braccio_description/urdf/camera_mount_model.urdf (robot description, URDF)
Before this commit: robot mounting, 1 links, 0 joints
Links:
- added link world
Joints:
- added joint world_joint: type fixed, parent world, child mount, origin xyz=0.0 0.0 0.0 rpy=0.0 0.0 0.0

File: braccio_description/urdf/xacros/_d435.urdf.xacro (robot description, xacro)
@@ -31,11 +31,11 @@
     <color rgba="0.5 0.5 0.5 1"/>
     </material>
-    <!-- camera body, with origin at bottom screw mount -->
-    <link name="${name}_bottom_screw_frame"/>
-    <!-- <joint name="${name}_joint" type="fixed">
+    <joint name="${name}_joint" type="fixed">
       <xacro:insert_block name="origin" />
       <parent link="${parent}"/>
       <child link="${name}_bottom_screw_frame" />
-    </joint> -->
+    </joint>
+     <!-- camera body, with origin at bottom screw mount -->
+    <link name="${name}_bottom_screw_frame"/>
     <joint name="${name}_link_joint" type="fixed">
       <origin xyz="0 ${d435_cam_depth_py} ${d435_cam_depth_pz}" rpy="0 0 0"/>
@@ -121,7 +121,3 @@
     <xacro:gazebo_d435 camera_name="${name}" reference_link="${name}_link" topics_ns="${topics_ns}" depth_optical_frame="${name}_depth_optical_frame" color_optical_frame="${name}_color_optical_frame" infrared1_optical_frame="${name}_left_ir_optical_frame" infrared2_optical_frame="${name}_right_ir_optical_frame" publish_pointcloud="${publish_pointcloud}"/>
   </xacro:macro>
-    <xacro:sensor_d435 parent="mount">
-          <!-- <origin xyz="0.0 0.0 0.5" rpy="0.0 0.0 0.0" /> -->
-          <origin xyz="0.0857 0.0000476009 -0.273184" rpy="0.0 0.0 0.0" />
-    </xacro:sensor_d435>
 </robot>
