Commit message: fixed robot self collision

File: braccio_description/urdf/xacros/braccio_model.urdf.xacro (robot description, xacro)
@@ -15,9 +15,15 @@
                         <cylinder length="0.01" radius=".053" />
                     </geometry>
-                    <material name="black" />
-                    <origin rpy="0 0 0" xyz="0 0 0.0" />
-                </visual>
-                <inertial>
-                    <origin rpy="0 0 0" xyz="0 0 0" />
+                    <!-- <material name="black" /> -->
+                    <origin rpy="0 0 0" xyz="0 0 0.020" />
+                </visual>
+                <collision>
+                    <geometry>
+                        <cylinder length="0.01" radius=".053" />
+                    </geometry>
+                    <origin rpy="0 0 0" xyz="0 0 0.020" />
+                </collision>
+                <inertial>
+                    <origin rpy="0 0 0" xyz="0 0 0.020" />
                     <mass value="2" />
                     <inertia ixx="0.015" ixy="0" ixz="0" iyy="0.00666666666667" iyz="0" izz="0.0216666666667" />
@@ -30,5 +36,5 @@
                     </geometry>
                     <material name="orange" />
-                    <origin rpy="0 0 3.1416" xyz="0 0.004 0" />
+                    <origin rpy="0 0 3.1416" xyz="0 0.004 0.023" />
                 </visual>
                 <collision>
@@ -36,8 +42,8 @@
                         <mesh filename="package://braccio_description/stl/braccio_base.stl" scale="0.001 0.001 0.001" />
                     </geometry>
-                    <origin rpy="0 0 3.1416" xyz="0 0.004 0" />
-                </collision>
-                <inertial>
-                    <origin rpy="0 0 3.1416" xyz="0 0.004 0" />
+                    <origin rpy="0 0 3.1416" xyz="0 0.004 0.023" />
+                </collision>
+                <inertial>
+                    <origin rpy="0 0 3.1416" xyz="0 0.004 0.023" />
                     <mass value="2" />
                     <inertia ixx="0.015" ixy="0" ixz="0" iyy="0.00666666666667" iyz="0" izz="0.0216666666667" />
@@ -302,7 +308,8 @@
                 <!-- <axis xyz="0 0 1"> -->
             <!-- </joint>  -->
-        <joint name="robot_joint" type="fixed" >
+        <joint name="robot_joint" type="contiuous" >
             <parent link="${parent}" />
             <child link="base_link" />
+            <axis xyz="0 0 -1" />
         </joint>
      </xacro:macro>

File: braccio_description/urdf/xacros/braccio_model_planning.urdf.xacro (robot description, xacro)
@@ -12,8 +12,14 @@
             </geometry>
             <material name="black" />
-            <origin rpy="0 0 0" xyz="0 0 0" />
-        </visual>
-        <inertial>
-            <origin rpy="0 0 0" xyz="0 0 0" />
+            <origin rpy="0 0 0" xyz="0 0 0.020" />
+        </visual>
+        <collision>
+            <geometry>
+                <cylinder length="0.01" radius=".053" />
+            </geometry>
+            <origin rpy="0 0 0" xyz="0 0 0.020" />
+        </collision>
+        <inertial>
+            <origin rpy="0 0 0" xyz="0 0 0.020" />
             <mass value="0.1"/>
             <inertia ixx="0.1" ixy="0.0" ixz="0.0" iyy="0.1" iyz="0.0" izz="0.1"/>
@@ -26,5 +32,5 @@
             </geometry>
             <material name="orange" />
-            <origin rpy="0 0 3.1416" xyz="0 0.004 0" />
+            <origin rpy="0 0 3.1416" xyz="0 0.004 0.023" />
         </visual>
         <collision>
@@ -32,8 +38,8 @@
                 <mesh filename="package://braccio_description/stl/braccio_base.stl" scale="0.001 0.001 0.001" />
             </geometry>
-            <origin rpy="0 0 0" xyz="0 0 0" />
-        </collision>
-        <inertial>
-            <origin rpy="0 0 0" xyz="0 0.002 0.031" />
+            <origin rpy="0 0 0" xyz="0 0 0.023" />
+        </collision>
+        <inertial>
+            <origin rpy="0 0 0" xyz="0 0.002 0.023" />
             <mass value="0.1"/>
             <inertia ixx="0.1" ixy="0.0" ixz="0.0" iyy="0.1" iyz="0.0" izz="0.1"/>
@@ -324,4 +330,5 @@
         <child link="base_link"/>
         <!-- <origin rpy="0.0 0.0 0.0" xyz="0.0 0.0 0.0"/> -->
+        <!-- <axis xyz="0 0 -1" /> -->
     </joint>
     </xacro:macro>

File: braccio_description/urdf/xacros/camera_mount_model.urdf.xacro (robot description, xacro)
@@ -4,5 +4,5 @@
         <link name="mount">
             <inertial>
-                <origin rpy="1.57 0 0" xyz="0 0.0 0" />
+                <origin rpy="1.57 0 0.78" xyz="0 0.0 0" />
                 <mass value="2" />
                 <inertia ixx="0.015" ixy="0" ixz="0" iyy="0.00666666666667" iyz="0" izz="0.0216666666667"/>
@@ -13,5 +13,5 @@
                 </geometry>
                 <material name="dark"/>
-                <origin rpy="1.57 0 0" xyz="0 0.0 0" />
+                <origin rpy="1.57 0 0.78" xyz="0 0.0 0" />
             </visual>
             <collision>
@@ -19,5 +19,5 @@
                     <mesh filename="package://braccio_description/stl/camera_mount.stl" scale="0.001 0.001 0.001"/>
                 </geometry>
-                <origin rpy="1.57 0 0" xyz="0 0.0 0" />
+                <origin rpy="1.57 0 0.78" xyz="0 0.0 0" />
             </collision>
         </link>
