Commit message: fixed camera orientation

File: braccio_description/urdf/xacros/braccio_model_planning.urdf.xacro (robot description, xacro)
@@ -325,10 +325,7 @@
         <material>Gazebo/Turquoise</material>
     </gazebo>
-    <!-- <link name="world"/> -->
     <joint name="robot_joint" type="fixed">
         <parent link="${parent}"/>
         <child link="base_link"/>
-        <!-- <origin rpy="0.0 0.0 0.0" xyz="0.0 0.0 0.0"/> -->
-        <!-- <axis xyz="0 0 -1" /> -->
     </joint>
     </xacro:macro>

File: braccio_description/urdf/xacros/camera_and_mount_and_braccio.urdf.xacro (robot description, xacro)
@@ -8,5 +8,5 @@
     </xacro:camera_mount>
     <xacro:sensor_d435 parent="mount">
-        <origin xyz="0.0 0.0 0.6" rpy="0.0 0.0 0.0" />
+        <origin xyz="0.0 0.0 0.6" rpy="0.0 1.0 1.10" />
     </xacro:sensor_d435>
     <xacro:kuka parent="mount">

File: braccio_description/urdf/xacros/camera_and_mount_and_braccio_planning.urdf.xacro (robot description, xacro)
@@ -8,5 +8,5 @@
     </xacro:camera_mount>
     <xacro:sensor_d435 parent="mount">
-        <origin xyz="0.0 0.0 0.6" rpy="0.0 0.0 0.0" />
+        <origin xyz="0.0 0.0 0.625" rpy="0.0 1.10 1.10" />
     </xacro:sensor_d435>
     <xacro:kr5 parent="mount">

File: braccio_description/urdf/xacros/camera_mount_model.urdf.xacro (robot description, xacro)
@@ -12,5 +12,5 @@
                     <mesh filename="package://braccio_description/stl/camera_mount.stl" scale="0.001 0.001 0.001"/>
                 </geometry>
-                <material name="dark"/>
+                <material name="white"/>
                 <origin rpy="1.57 0 0.78" xyz="0 0.0 0" />
             </visual>
