Commit message: added mount link to manipulator.srdf

File: braccio_description/urdf/xacros/camera_mount_model.urdf.xacro (robot description, xacro)
@@ -22,7 +22,8 @@
             </collision>
         </link>
-        <joint name="mount_joint" type="fixed" >
+        <joint name="mount_joint" type="continuous" >
             <parent link="${parent}" />
             <child link="mount" />
+            <axis xyz="0 0 -1" />
         </joint>
     </xacro:macro>
